File: Hardware/Alarm_Clock_PCB/Alarm_Clock_PCB.kicad_sch (KiCad schematic)
At the start: 19 parts, among them J1 Conn_01x20_Socket, J2 Conn_01x20_Socket, J3 Conn_01x04_Socket, J4 Conn_01x06_Socket, J5 Screw_Terminal_01x02, J6 Screw_Terminal_01x02, J7 Screw_Terminal_01x02, J8 Screw_Terminal_01x02, Q1 Q_NMOS

Commit message: Did some footprint stuff
Got some footprints sorted out.
Parts:
- J1, J2, J3, J4: footprint (none) -> Connector_PinHeader_1.00mm:PinHeader_1x20_P1.00mm_Vertical
- J5, Q1: footprint (none) -> Package_TO_SOT_SMD:SOT-23-5_HandSoldering
- LS1: footprint TMB12A05 -> 00-footprint-library:TMB12A05
Changed lines of the file:
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@@
 			)
 		)
-		(property "Footprint" ""
+		(property "Footprint" "Connector_PinHeader_1.00mm:PinHeader_1x20_P1.00mm_Vertical"
 			(at 72.39 59.69 0)
 			(effects
@@
 			)
 		)
-		(property "Footprint" ""
+		(property "Footprint" "Package_TO_SOT_SMD:SOT-23-5_HandSoldering"
 			(at 255.27 46.99 0)
 			(effects
@@
 			)
 		)
-		(property "Footprint" ""
+		(property "Footprint" "Connector_PinHeader_1.00mm:PinHeader_1x20_P1.00mm_Vertical"
 			(at 195.58 83.82 0)
 			(effects
@@
 			)
 		)
-		(property "Footprint" "TMB12A05"
+		(property "Footprint" "00-footprint-library:TMB12A05"
 			(at 264.16 163.5 0)
 			(effects
@@
 			)
 		)
-		(property "Footprint" ""
+		(property "Footprint" "Connector_PinHeader_1.00mm:PinHeader_1x20_P1.00mm_Vertical"
 			(at 96.52 59.69 0)
 			(effects
@@
 			)
 		)
-		(property "Footprint" ""
+		(property "Footprint" "Connector_PinHeader_1.00mm:PinHeader_1x20_P1.00mm_Vertical"
 			(at 185.42 43.18 0)
 			(effects
@@
 			)
 		)
-		(property "Footprint" ""
+		(property "Footprint" "Package_TO_SOT_SMD:SOT-23-5_HandSoldering"
 			(at 95.25 143.51 0)
 			(effects

Commit message: Did Initial Layout Work
Worked on finishing on choosing footprints and also did initial footprint layout. Also began to look into constraints on Kicad.
Parts:
- removed Q1: Q_NMOS, Package_TO_SOT_SMD:SOT-23-5_HandSoldering, symbol Device:Q_NMOS
- added H1, H2, H3, H4: MountingHole, MountingHole:MountingHole_2.2mm_M2, symbol Mechanical:MountingHole
- added Q1: NMOS, Package_TO_SOT_SMD:SOT-23-3, symbol Simulation_SPICE:NMOS
- J3: footprint Connector_PinHeader_1.00mm:PinHeader_1x20_P1.00mm_Vertical -> Connector_PinHeader_1.00mm:PinHeader_1x04_P1.00mm_Vertical
- J4: footprint Connector_PinHeader_1.00mm:PinHeader_1x20_P1.00mm_Vertical -> Connector_PinHeader_1.00mm:PinHeader_1x06_P1.00mm_Vertical
- J5: footprint Package_TO_SOT_SMD:SOT-23-5_HandSoldering -> 00-footprint-library:CONN_OSTVN02A150_OST
- J6, J7, J8: footprint (none) -> 00-footprint-library:CONN_OSTVN02A150_OST
Connections:
- net GP10: now also J1.14 (Pin_14)
- net GP11: now also J1.15 (Pin_15)
- net GP12: now also J1.16 (Pin_16)
- net GP13: now also J1.17 (Pin_17)
- net GP14: now also J1.19 (Pin_19)
- net VBUS: now also Q1.1 (D)
- net at R9.1: now also Q1.2 (G)
- net at LS1.1 (+): now also Q1.3 (S)
- no-connect marks 2 -> 25
Other:
- note added: "Mounting Holes"
