File: Hardware/Alarm_Clock_PCB/Alarm_Clock_PCB.kicad_pcb (KiCad board)
At the start: 2 copper layers, 55 x 38 mm, 23 parts, among them J1 Conn_01x20_Socket, J2 Conn_01x20_Socket, J3 Conn_01x04_Socket, J4 Conn_01x06_Socket, J5 Screw_Terminal_01x02, J6 Screw_Terminal_01x02, J7 Screw_Terminal_01x02, J8 Screw_Terminal_01x02, Q1 NMOS

Commit message: Finished Routing on PCB
Finished off routing and cleared off all the errors, the only thing left to do on the PCB is getting Gerber files for ordering.
Routing:
- net VBUS: track 0.00 -> 64.6 mm
- net +3.3V: track 0.00 -> 36.4 mm, vias 0 -> 4
- net Net-(J8-Pin_1): track 0.00 -> 27.0 mm
- net Net-(J7-Pin_1): track 0.00 -> 18.6 mm
- net Net-(J5-Pin_1): track 0.00 -> 15.4 mm
- net GND: track 0.00 -> 14.4 mm
- net Net-(J6-Pin_1): track 0.00 -> 12.9 mm
- net Net-(LS1-+): track 0.00 -> 8.55 mm
- net GP5: track 0.00 -> 7.45 mm
- net GP4: track 0.00 -> 7.45 mm
- net Net-(Q1-G): track 0.00 -> 3.32 mm
- net GP14: track 0.00 -> 2.74 mm
- net GP13: track 0.00 -> 1.89 mm
- net GP10: track 0.00 -> 1.87 mm
- net GP12: track 0.00 -> 1.82 mm
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- added copper zone on B.Cu, net GND
- removed copper zone on B.Cu, net (none)
