File: Hardware/Alarm_Clock_PCB/Alarm_Clock_PCB.kicad_pcb (KiCad board)
At the start: 2 copper layers, 55 x 38 mm, 23 parts, among them J1 Conn_01x20_Socket, J2 Conn_01x20_Socket, J3 Conn_01x04_Socket, J4 Conn_01x06_Socket, J5 Screw_Terminal_01x02, J6 Screw_Terminal_01x02, J7 Screw_Terminal_01x02, J8 Screw_Terminal_01x02, Q1 NMOS

Commit message: Fixed a issue with the Mosfet for the buzzer.
NMOS was place on the high side but should be place on the low side.
Parts:
- moved LS1 9.91 mm to (107.3, 83.0), turned to -90 degrees
- moved Q1 4.83 mm to (108.1, 92.8), turned to -90 degrees
Connections:
- LS1 pad 1: Net-(LS1-+) -> VBUS
- LS1 pad 2: GND -> Net-(LS1--)
- Q1 pad 1: VBUS -> Net-(LS1--)
- Q1 pad 3: Net-(LS1-+) -> GND
Routing:
- net Net-(LS1--): track 0.00 -> 11.0 mm
- net Net-(LS1-+): track 8.55 -> 0.00 mm
- net VBUS: track 64.6 -> 70.8 mm
- net Net-(Q1-G): track 3.32 -> 7.84 mm
- net GND: track 14.4 -> 15.0 mm, vias 0 -> 1
